Commit message: fix: box collisions for SO-101 jaws so convex hulls don't fill the gap
Co-Authored-By: Claude Sonnet 5.5 <noreply@anthropic.com>
Claude-Session: https://claude.ai/code/session_01HmKGXjFrjvGk7fW4QkXQxY

File: assets/so101/so101_new_calib.urdf (robot description, URDF)
Before this commit: robot so101_new_calib, 8 links, 7 joints
Links:
- link gripper_link: geometry collision box size=0.02658 0.02377 0.05931; collision box size=0.06520 0.05200 0.04543
- link moving_jaw_so101_v1_link: geometry collision box size=0.01883 0.05011 0.01902; collision box size=0.02000 0.03971 0.04800
